File: Hardware/LMG1025_Flasher_Shield.brd (EAGLE design)
At the start: 48.6 x 53.3 mm, 43 parts, among them K1 TLP3475R(TP,F, K2 TLP3475R(TP,F, K3 TLP3475R(TP,F, K4 TLP3475R(TP,F, U1 DS1023-25, U2 LMG1025, U3 MAX-M8, U4 74AHCT1G125DBV

Commit message: Added the BOM
Parts:
- D2: value CD0603-B00340 -> 0.5A/40V/420mV; device SamacSys_Parts:DIOM179X85N -> SparkFun-DiscreteSemi:SOD-323
Connections:
- net 3.3V: now also D2.C; no longer D2.1
- net RX: now also D2.A; no longer D2.2
Routing:
- net GND: track 36.1 -> 35.4 mm
Changed lines of the file:
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@@
 <?xml version="1.0" encoding="utf-8"?>
 <!DOCTYPE eagle SYSTEM "eagle.dtd">
-<eagle version="9.5.2">
+<eagle version="9.6.0">
 <drawing>
 <settings>
@@
 <attribute name="NAME" x="38.735" y="32.131" size="0.8128" layer="25" ratio="15" rot="R270"/>
 </element>
-<element name="D2" library="SamacSys_Parts" package="DIOM179X85N" value="CD0603-B00340" x="29.21" y="23.495" smashed="yes" rot="R270">
-<attribute name="ARROW_PART_NUMBER" value="CD0603-B00340" x="29.21" y="27.305" size="1.778" layer="27" rot="R270" display="off"/>
-<attribute name="DESCRIPTION" value="Diode Schottky Signal 45V 30mA 0603 Bourns CD0603-B00340, SMT Schottky Diode, 45V 30mA, 2-Pin 0603" x="29.21" y="27.305" size="1.778" layer="27" rot="R270" display="off"/>
-<attribute name="HEIGHT" value="0.85mm" x="29.21" y="27.305" size="1.778" layer="27" rot="R270" display="off"/>
-<attribute name="MANUFACTURER_NAME" value="Bourns" x="29.21" y="27.305" size="1.778" layer="27" rot="R270" display="off"/>
-<attribute name="MANUFACTURER_PART_NUMBER" value="CD0603-B00340" x="29.21" y="27.305" size="1.778" layer="27" rot="R270" display="off"/>
-<attribute name="NAME" x="29.337" y="20.828" size="0.8128" layer="25" ratio="15" rot="R270" align="center"/>
-</element>
 <element name="U3" library="ubloxLib" package="MAX-M8" value="MAX-M8" x="35.56" y="21.59" smashed="yes" rot="R90"/>
 <element name="R11" library="microbuilder" package="0805-NO" value="10 ohm" x="28.829" y="14.605" smashed="yes" rot="R90">
@@
 <element name="TP3" library="SparkFun-Connectors" package="1X01_NO_SILK" value="TEST-POINTPOGO_PTH" x="25.4" y="40.64" smashed="yes">
 <attribute name="NAME" x="24.384" y="41.91" size="0.8128" layer="25" font="vector" ratio="15"/>
+</element>
+<element name="D2" library="SparkFun-DiscreteSemi" package="SOD-323" value="0.5A/40V/420mV" x="29.21" y="23.495" smashed="yes" rot="SR270">
+<attribute name="NAME" x="29.591" y="26.162" size="0.8128" layer="25" font="vector" ratio="18" rot="SR90" align="bottom-center"/>
+<attribute name="PROD_ID" value="DIO-10955" x="29.21" y="23.495" size="1.778" layer="27" rot="SR270" display="off"/>
 </element>
 </elements>
@@
 <wire x1="30.248" y1="17.04" x2="30.226" y2="17.018" width="0.4064" layer="1"/>
 <via x="30.226" y="17.018" extent="1-16" drill="0.4"/>
-<wire x1="11.684" y1="42.5323" x2="11.684" y2="43.307" width="0.4064" layer="1"/>
 <wire x1="39.96" y1="26.54" x2="41.272" y2="26.54" width="0.4064" layer="1"/>
 <wire x1="41.272" y1="26.54" x2="41.275" y2="26.543" width="0.4064" layer="1"/>
@@
 <signal name="3.3V">
 <contactref element="PCB1" pad="3.3V"/>
-<contactref element="D2" pad="1"/>
 <contactref element="D1" pad="A"/>
 <contactref element="U3" pad="7_VCC_IO"/>
@@
 <contactref element="C7" pad="1"/>
 <via x="27.559" y="24.257" extent="1-16" drill="0.4"/>
-<wire x1="27.559" y1="24.257" x2="29.172" y2="24.257" width="0.8128" layer="1"/>
-<wire x1="29.172" y1="24.257" x2="29.21" y2="24.295" width="0.8128" layer="1"/>
-<wire x1="29.21" y1="24.295" x2="31.788" y2="24.295" width="0.8128" layer="1"/>
+<wire x1="29.172" y1="24.257" x2="27.559" y2="24.257" width="0.8128" layer="1"/>
 <wire x1="32.31" y1="24.817" x2="32.31" y2="26.54" width="0.8128" layer="1"/>
-<wire x1="31.788" y1="24.295" x2="32.31" y2="24.817" width="0.8128" layer="1"/>
+<wire x1="32.31" y1="24.817" x2="31.788" y2="24.295" width="0.8128" layer="1"/>
 <wire x1="33.41" y1="26.54" x2="32.31" y2="26.54" width="0.8128" layer="1"/>
 <wire x1="32.319" y1="29.337" x2="32.31" y2="29.328" width="0.8128" layer="1"/>
@@
 <wire x1="18.796" y1="21.463" x2="18.796" y2="9.017" width="1.016" layer="1"/>
 <wire x1="16.136" y1="9.017" x2="18.796" y2="9.017" width="0.4064" layer="1"/>
+<contactref element="D2" pad="C"/>
+<wire x1="29.21" y1="24.645" x2="29.21" y2="24.295" width="0.8128" layer="1"/>
+<wire x1="29.21" y1="24.295" x2="29.172" y2="24.257" width="0.8128" layer="1"/>
+<wire x1="31.788" y1="24.295" x2="29.21" y2="24.295" width="0.8128" layer="1"/>
 </signal>
 <signal name="TX">
@@
 <signal name="RX">
 <contactref element="R13" pad="1"/>
-<contactref element="D2" pad="2"/>
 <contactref element="U3" pad="3_RXD"/>
 <wire x1="38.1" y1="44.362" x2="41.275" y2="41.187" width="0.4064" layer="1"/>
@@
 <wire x1="40.894" y1="29.464" x2="38.481" y2="29.464" width="0.4064" layer="1"/>
 <wire x1="38.481" y1="29.464" x2="37.81" y2="28.793" width="0.4064" layer="1"/>
-<wire x1="29.21" y1="22.695" x2="36.665" y2="22.695" width="0.4064" layer="1"/>
-<wire x1="37.81" y1="23.84" x2="37.81" y2="26.54" width="0.4064" layer="1"/>
-<wire x1="36.665" y1="22.695" x2="37.81" y2="23.84" width="0.4064" layer="1"/>
+<wire x1="37.81" y1="26.54" x2="37.81" y2="23.84" width="0.4064" layer="1"/>
+<contactref element="D2" pad="A"/>
+<wire x1="36.315" y1="22.345" x2="29.21" y2="22.345" width="0.4064" layer="1"/>
+<wire x1="37.81" y1="23.84" x2="36.315" y2="22.345" width="0.4064" layer="1"/>
 </signal>
 <signal name="TP">
